File: pcb/Numpadv1/.history/Numpadv1.kicad_pcb (KiCad board)
At the start: 2 copper layers, 104.8 x 100 mm, 40 parts, among them J1 OLED_128x32, SW1 RotaryEncoder_Switch, SW2 Switch, SW3 Switch, SW4 Switch, U1 RP2040_Zero

Commit message: PCB Manufacturing Files
Parts:
- added H1: ~, ScottoKeebs_Scotto:Standoff_M2x4mm, B.Cu at (83.2, 67.3)
- added H2: ~, ScottoKeebs_Scotto:Standoff_M2x4mm, B.Cu at (83.2, 124.5)
- added H3: ~, ScottoKeebs_Scotto:Standoff_M2x4mm, B.Cu at (140.3, 105.4)
- added H4: ~, ScottoKeebs_Scotto:Standoff_M2x4mm, F.Cu at (1.62, 1.62)
- moved SW1 45.1 mm to (153.5, 85.0)
- moved J1 21.4 mm to (159.4, 99.0)
- moved U1 1.91 mm to (154.1, 60.2)
Routing:
- net /Row 4: track 0.00 -> 120.1 mm
- net /Row 3: track 0.45 -> 112.9 mm
- net /Row 2: track 0.00 -> 104.1 mm
- net /Col 0: track 89.7 -> 186.8 mm
- net /Row 1: track 0.00 -> 91.7 mm
- net /Col 1: track 57.1 -> 143.5 mm
- net /GND: track 0.00 -> 68.0 mm
- net /Col 2: track 76.2 -> 143.4 mm
- net /Col 3: track 66.4 -> 117.5 mm, vias 0 -> 2
- net /3V3: track 0.00 -> 47.9 mm
- net /I2C0 SCL: track 0.00 -> 32.2 mm
- net /I2C0 SDA: track 0.00 -> 31.6 mm
- net /Row 0: track 57.2 -> 82.9 mm
- net /GP10: track 0.00 -> 19.0 mm
- net /GP11: track 0.00 -> 14.0 mm
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- added copper zone on B.Cu, net /GND
- added copper zone on F.Cu, net /GND
