File: pcb/Numpadv1/.history/Numpadv1.kicad_sch (KiCad schematic)
At the start: 37 parts, among them J1 OLED_128x32, SW1 RotaryEncoder_Switch, U1 RP2040_Zero

Commit message: PCB Completed (for now)
Parts:
- added H1, H2, H3: (no value), ScottoKeebs_Scotto:Standoff_M2x4mm, symbol ScottoKeebs:Placeholder_Mounting_Hole
- added SW2, SW3, SW4: Switch, ScottoKeebs_Stabilizer:Stabilizer_MX_2.00u, symbol ScottoKeebs:Placeholder_Switch
- S1, S10, S11, S12, S13, S14, S15, S2, S3, S4, S6, S7, S8, S9: footprint ScottoKeebs_MX:MX_PCB_1.00u -> ScottoKeebs_Hotswap:Hotswap_MX_1.00u
- S16, S17: footprint Button_Switch_Keyboard:SW_Cherry_MX_2.00u_Vertical_PCB -> ScottoKeebs_Hotswap:Hotswap_MX_2.00u_90deg
- S5: footprint Button_Switch_Keyboard:SW_Cherry_MX_2.00u_PCB -> ScottoKeebs_Hotswap:Hotswap_MX_2.00u
Connections:
- net Col 0: now also S5.1; no longer S5.2
- net Col 3: now also S16.1, S17.1; no longer S16.2, S17.2
- net Row 1: no longer D16.1 (K)
- net Row 2: now also D16.1 (K)
- net Row 3: no longer D17.1 (K)
- net Row 4: now also D17.1 (K)
- net at D17.2 (A): now also S17.2; no longer S17.1
- net at D5.2 (A): now also S5.2; no longer S5.1
- net at D16.2 (A): now also S16.2; no longer S16.1
Other:
- moved on the sheet: D16, D17, S16, S17, S5

Commit message: PCB Manufacturing Files
Other:
- moved on the sheet: SW2, SW3, SW4
Changed lines of the file:
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@@
 	(symbol
 		(lib_id "ScottoKeebs:Placeholder_Switch")
-		(at 167.64 113.03 0)
+		(at 185.42 111.76 0)
 		(unit 1)
 		(body_style 1)
@@
 		(fields_autoplaced yes)
 		(property "Reference" "SW3"
-			(at 167.64 105.41 0)
+			(at 185.42 104.14 0)
 			(show_name no)
 			(do_not_autoplace no)
@@
 		)
 		(property "Value" "Switch"
-			(at 167.64 107.95 0)
+			(at 185.42 106.68 0)
 			(show_name no)
 			(do_not_autoplace no)
@@
 		)
 		(property "Footprint" "ScottoKeebs_Stabilizer:Stabilizer_MX_2.00u"
-			(at 167.64 107.95 0)
-			(hide yes)
-			(show_name no)
-			(do_not_autoplace no)
-			(effects
-				(font
-					(size 1.27 1.27)
-				)
-			)
-		)
-		(property "Datasheet" ""
-			(at 167.64 107.95 0)
+			(at 185.42 106.68 0)
+			(hide yes)
+			(show_name no)
+			(do_not_autoplace no)
+			(effects
+				(font
+					(size 1.27 1.27)
+				)
+			)
+		)
+		(property "Datasheet" ""
+			(at 185.42 106.68 0)
 			(hide yes)
 			(show_name no)
@@
 		)
 		(property "Description" "Push button switch, generic, two pins"
-			(at 167.64 113.03 0)
+			(at 185.42 111.76 0)
 			(hide yes)
 			(show_name no)
@@
 	(symbol
 		(lib_id "ScottoKeebs:Placeholder_Switch")
-		(at 118.11 125.73 0)
+		(at 121.92 143.51 0)
 		(unit 1)
 		(body_style 1)
@@
 		(fields_autoplaced yes)
 		(property "Reference" "SW2"
-			(at 118.11 118.11 0)
+			(at 121.92 135.89 0)
 			(show_name no)
 			(do_not_autoplace no)
@@
 		)
 		(property "Value" "Switch"
-			(at 118.11 120.65 0)
+			(at 121.92 138.43 0)
 			(show_name no)
 			(do_not_autoplace no)
@@
 		)
 		(property "Footprint" "ScottoKeebs_Stabilizer:Stabilizer_MX_2.00u"
-			(at 118.11 120.65 0)
-			(hide yes)
-			(show_name no)
-			(do_not_autoplace no)
-			(effects
-				(font
-					(size 1.27 1.27)
-				)
-			)
-		)
-		(property "Datasheet" ""
-			(at 118.11 120.65 0)
+			(at 121.92 138.43 0)
+			(hide yes)
+			(show_name no)
+			(do_not_autoplace no)
+			(effects
+				(font
+					(size 1.27 1.27)
+				)
+			)
+		)
+		(property "Datasheet" ""
+			(at 121.92 138.43 0)
 			(hide yes)
 			(show_name no)
@@
 		)
 		(property "Description" "Push button switch, generic, two pins"
-			(at 118.11 125.73 0)
+			(at 121.92 143.51 0)
 			(hide yes)
 			(show_name no)
@@
 	(symbol
 		(lib_id "ScottoKeebs:Placeholder_Switch")
-		(at 167.64 85.09 0)
+		(at 185.42 83.82 0)
 		(unit 1)
 		(body_style 1)
@@
 		(fields_autoplaced yes)
 		(property "Reference" "SW4"
-			(at 167.64 77.47 0)
+			(at 185.42 76.2 0)
 			(show_name no)
 			(do_not_autoplace no)
@@
 		)
 		(property "Value" "Switch"
-			(at 167.64 80.01 0)
+			(at 185.42 78.74 0)
 			(show_name no)
 			(do_not_autoplace no)
@@
 		)
 		(property "Footprint" "ScottoKeebs_Stabilizer:Stabilizer_MX_2.00u"
-			(at 167.64 80.01 0)
-			(hide yes)
-			(show_name no)
-			(do_not_autoplace no)
-			(effects
-				(font
-					(size 1.27 1.27)
-				)
-			)
-		)
-		(property "Datasheet" ""
-			(at 167.64 80.01 0)
+			(at 185.42 78.74 0)
+			(hide yes)
+			(show_name no)
+			(do_not_autoplace no)
+			(effects
+				(font
+					(size 1.27 1.27)
+				)
+			)
+		)
+		(property "Datasheet" ""
+			(at 185.42 78.74 0)
 			(hide yes)
 			(show_name no)
@@
 		)
 		(property "Description" "Push button switch, generic, two pins"
-			(at 167.64 85.09 0)
-			(hide yes)
-			(show_name no)
+			(at 185.42 83.82 0)
+			(hide yes)
+			(show_name no)
