File: pcb/Numpadv1/.history/Numpadv1.kicad_sch (KiCad schematic)
At the start: 43 parts, among them J1 OLED_128x32, SW1 RotaryEncoder_Switch, SW2 Switch, SW3 Switch, SW4 Switch, U1 RP2040_Zero

Commit message: Routing Fixed
Connections:
- net GP10: now also U1.11 (10); no longer U1.10 (9)
- net GP11: now also U1.12 (11); no longer U1.11 (10)
- net GP14: now also U1.15 (14); no longer U1.14 (13)
- net I2C0 SCL: now also U1.14 (13); no longer U1.13 (12)
- net I2C0 SDA: now also U1.13 (12); no longer U1.12 (11)
Changed lines of the file:
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@@
-	(wire
-		(pts
-			(xy 73.66 67.31) (xy 73.66 63.5)
-		)
-		(stroke
-			(width 0)
-			(type default)
-		)
-	)
 	(wire
 		(pts
@@
 	(wire
 		(pts
-			(xy 81.28 67.31) (xy 81.28 63.5)
-		)
-		(stroke
-			(width 0)
-			(type default)
-		)
-	)
-	(wire
-		(pts
 			(xy 119.38 113.03) (xy 139.7 113.03)
 		)
@@
 	(wire
 		(pts
-			(xy 78.74 67.31) (xy 78.74 63.5)
-		)
-		(stroke
-			(width 0)
-			(type default)
-		)
-	)
-	(wire
-		(pts
 			(xy 119.38 99.06) (xy 129.54 99.06)
 		)
@@
 	(wire
 		(pts
-			(xy 71.12 67.31) (xy 71.12 63.5)
-		)
-		(stroke
-			(width 0)
-			(type default)
-		)
-	)
-	(wire
-		(pts
 			(xy 139.7 85.09) (xy 149.86 85.09)
 		)
@@
 	(wire
 		(pts
-			(xy 76.2 67.31) (xy 76.2 63.5)
-		)
-		(stroke
-			(width 0)
-			(type default)
-		)
-	)
-	(wire
-		(pts
 			(xy 91.44 45.72) (xy 88.9 45.72)
 		)
@@
 	)
 	(label "I2C0 SDA"
-		(at 76.2 67.31 270)
+		(at 73.66 63.5 270)
 		(effects
 			(font
@@
 	)
 	(label "GP10"
-		(at 81.28 67.31 270)
+		(at 78.74 63.5 270)
 		(effects
 			(font
@@
 	)
 	(label "GP11"
-		(at 78.74 67.31 270)
+		(at 76.2 63.5 270)
 		(effects
 			(font
@@
 	)
 	(label "GP14"
-		(at 71.12 67.31 270)
+		(at 63.5 58.42 180)
 		(effects
 			(font
@@
 	)
 	(label "I2C0 SCL"
-		(at 73.66 67.31 270)
-		(effects
-			(font
+		(at 71.12 63.5 270)
+		(effects
+			(font
