File: pcb/Numpadv1/Numpadv1.kicad_pcb (KiCad board)
At the start: 2 copper layers, 104.8 x 100 mm, 44 parts, among them J1 OLED_128x32, SW1 RotaryEncoder_Switch, SW2 Switch, SW3 Switch, SW4 Switch, U1 RP2040_Zero

Commit message: Routing Fixed
Connections:
- U1 pad 10: /GP10 -> unconnected-(U1-9-Pad10)
- U1 pad 11: /GP11 -> /GP10
- U1 pad 12: /I2C0 SDA -> /GP11
- U1 pad 13: /I2C0 SCL -> /I2C0 SDA
- U1 pad 14: /GP14 -> /I2C0 SCL
- U1 pad 15: unconnected-(U1-14-Pad15) -> /GP14
Routing:
- net /GP10: track 19.0 -> 20.1 mm
- net /I2C0 SDA: track 31.6 -> 32.7 mm
- net /GP11: track 14.0 -> 15.0 mm
- net /GP14: track 13.2 -> 12.2 mm
- net /I2C0 SCL: track 32.2 -> 32.7 mm, vias 0 -> 1
Changed lines of the file:
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@@
 			(layers "*.Cu" "*.Mask")
 			(remove_unused_layers no)
-			(net "/GP10")
+			(net "unconnected-(U1-9-Pad10)")
 			(pinfunction "9_10")
 			(pintype "bidirectional")
@@
 			(layers "*.Cu" "*.Mask")
 			(remove_unused_layers no)
-			(net "/GP11")
+			(net "/GP10")
 			(pinfunction "10_11")
 			(pintype "bidirectional")
@@
 			(layers "*.Cu" "*.Mask")
 			(remove_unused_layers no)
-			(net "/I2C0 SDA")
+			(net "/GP11")
 			(pinfunction "11_12")
 			(pintype "bidirectional")
@@
 			(layers "*.Cu" "*.Mask")
 			(remove_unused_layers no)
-			(net "/I2C0 SCL")
+			(net "/I2C0 SDA")
 			(pinfunction "12_13")
 			(pintype "bidirectional")
@@
 			(layers "*.Cu" "*.Mask")
 			(remove_unused_layers no)
-			(net "/GP14")
+			(net "/I2C0 SCL")
 			(pinfunction "13_14")
 			(pintype "bidirectional")
@@
 			(layers "*.Cu" "*.Mask")
 			(remove_unused_layers no)
-			(net "unconnected-(U1-14-Pad15)")
+			(net "/GP14")
 			(pinfunction "14_15")
 			(pintype "bidirectional")
@@
 	)
 	(segment
-		(start 159.1775 70.32625)
-		(end 162.27875 73.4275)
+		(start 156.6375 74.0875)
+		(end 156.6375 70.32625)
 		(width 0.2)
-		(layer "B.Cu")
+		(layer "F.Cu")
 		(net "/GP10")
 	)
 	(segment
-		(start 162.27875 86.21625)
-		(end 160.97875 87.51625)
+		(start 162.27875 79.72875)
+		(end 156.6375 74.0875)
 		(width 0.2)
-		(layer "B.Cu")
+		(layer "F.Cu")
 		(net "/GP10")
 	)
 	(segment
-		(start 162.27875 73.4275)
-		(end 162.27875 86.21625)
+		(start 162.27875 86.21625)
+		(end 162.27875 79.72875)
 		(width 0.2)
-		(layer "B.Cu")
+		(layer "F.Cu")
 		(net "/GP10")
 	)
 	(segment
-		(start 159.385 73.07375)
-		(end 156.6375 70.32625)
+		(start 160.97875 87.51625)
+		(end 162.27875 86.21625)
 		(width 0.2)
-		(layer "B.Cu")
-		(net "/GP11")
+		(layer "F.Cu")
+		(net "/GP10")
 	)
 	(segment
-		(start 159.385 80.9225)
-		(end 159.385 73.07375)
+		(start 154.0975 75.635)
+		(end 160.97875 82.51625)
 		(width 0.2)
-		(layer "B.Cu")
+		(layer "F.Cu")
 		(net "/GP11")
 	)
 	(segment
-		(start 160.97875 82.51625)
-		(end 159.385 80.9225)
+		(start 154.0975 70.32625)
+		(end 154.0975 75.635)
 		(width 0.2)
-		(layer "B.Cu")
+		(layer "F.Cu")
 		(net "/GP11")
 	)
@@
 	)
 	(segment
-		(start 149.585 90.8475)
-		(end 149.585 100.6475)
+		(start 146.47875 87.51625)
+		(end 146.47875 87.74125)
 		(width 0.2)
 		(layer "B.Cu")
@@
 	)
 	(segment
-		(start 146.47875 87.51625)
-		(end 146.47875 87.74125)
+		(start 143.31625 66.71)
+		(end 143.31625 55.7075)
 		(width 0.2)
 		(layer "B.Cu")
@@
 	)
 	(segment
-		(start 143.31625 66.71)
-		(end 143.31625 55.7075)
+		(start 147.47875 98.54125)
+		(end 149.585 100.6475)
+		(width 0.2)
+		(layer "B.Cu")
+		(net "/GND")
+	)
+	(segment
+		(start 146.47875 87.74125)
+		(end 147.47875 88.74125)
 		(width 0.2)
 		(layer "B.Cu")
@@
 	)
 	(segment
-		(start 146.47875 87.51625)
-		(end 142.71625 83.75375)
+		(start 147.47875 88.74125)
+		(end 147.47875 98.54125)
 		(width 0.2)
 		(layer "B.Cu")
@@
 	)
 	(segment
-		(start 146.47875 87.74125)
-		(end 149.585 90.8475)
+		(start 146.47875 87.51625)
+		(end 142.71625 83.75375)
 		(width 0.2)
 		(layer "B.Cu")
@@
 	(segment
 		(start 146.47875 82.51625)
-		(end 149.0175 79.9775)
+		(end 146.47875 70.3275)
 		(width 0.2)
 		(layer "B.Cu")
@@
 	)
 	(segment
-		(start 149.0175 79.9775)
-		(end 149.0175 70.32625)
+		(start 146.47875 70.3275)
+		(end 146.4775 70.32625)
 		(width 0.2)
 		(layer "B.Cu")
@@
 	(segment
 		(start 157.205 100.6475)
-		(end 157.205 73.43375)
+		(end 151.5575 95)
 		(width 0.2)
 		(layer "B.Cu")
@@
 	)
 	(segment
-		(start 157.205 73.43375)
-		(end 154.0975 70.32625)
+		(start 151.5575 95)
+		(end 151.5575 70.32625)
 		(width 0.2)
 		(layer "B.Cu")
@@
 	)
 	(segment
-		(start 155.37875 99.93375)
-		(end 155.37875 74.1475)
+		(start 149.225 90.17)
+		(end 149.225 95.2075)
 		(width 0.2)
-		(layer "B.Cu")
+		(layer "F.Cu")
 		(net "/I2C0 SCL")
 	)
 	(segment
-		(start 155.37875 74.1475)
-		(end 151.5575 70.32625)
+		(start 149.225 95.2075)
+		(end 154.665 100.6475)
+		(width 0.2)
+		(layer "F.Cu")
+		(net "/I2C0 SCL")
+	)
+	(via
+		(at 149.225 90.17)
+		(size 0.6)
+		(drill 0.3)
+		(layers "F.Cu" "B.Cu")
+		(net "/I2C0 SCL")
+	)
+	(segment
+		(start 149.225 70.53375)
+		(end 149.0175 70.32625)
 		(width 0.2)
 		(layer "B.Cu")
@@
 	)
 	(segment
-		(start 154.665 100.6475)
-		(end 155.37875 99.93375)
+		(start 149.225 90.17)
+		(end 149.225 70.53375)
 		(width 0.2)
 		(layer "B.Cu")
